File: BGKYPRO_Gasket_Plate.kicad_pcb (KiCad board)
At the start: 2 copper layers, 294 x 105 mm, 0 parts

Commit message: brush up
Other:
- board size 294 x 105 mm -> 294 x 104 mm

Commit message: fix
Other:
- board size 294 x 104 mm -> 295 x 104 mm
